File: pcb/wcp52-input.sch (KiCad schematic (older format))
At the start: 18 parts, among them J1 5V, J2 -5V, J3 IN1, J4 IN2, J5 CTRL, J6 PHASEREF, J7 5V, Q1 PMV160UP, Q2 2N7002

Commit message: Associated parts with footprints
Parts:
- C1, C2: footprint (none) -> IPC7351-Nominal:CAPC3216X70
- C10, C11: footprint (none) -> IPC7351-Nominal:CAPC1005X55
- E1, E2: footprint (none) -> IPC7351-Nominal:INDC1005X60; Manuf (none) -> Value; PN (none) -> BK1005HS601-T
- J1, J2, J5, J7: footprint (none) -> conn:CONN_2-SIL
- J3, J4, J6: footprint (none) -> conn:CONN-2_CONSMA001-SMD-G
- Q1, Q2: footprint (none) -> IPC-semi-nominal:SOT-23
- R5, R6: footprint (none) -> IPC7351-Nominal:RESC1005X40
Changed lines of the file:
@@
 F 0 "J4" H 800 4000 50  0000 C CNN
 F 1 "IN2" H 800 3900 50  0000 C CNN
-F 2 "" H 800 3800 50  0000 C CNN
+F 2 "conn:CONN-2_CONSMA001-SMD-G" H 800 3800 50  0001 C CNN
 F 3 "" H 800 3800 50  0000 C CNN
 	1    800  3800
 	1    0    0    -1
-$EndComp
-$Comp
-L BEAD E1
-U 1 1 54565FC7
-P 1900 2000
-F 0 "E1" H 1900 1750 50  0000 C CNN
-F 1 "600" H 1900 1850 50  0000 C CNN
-F 2 "" H 1900 2050 60  0000 C CNN
-F 3 "" H 1900 2050 60  0000 C CNN
-	1    1900 2000
-	1    0    0    1
 $EndComp
 $Comp
@@
 F 0 "J1" H 800 2200 50  0000 C CNN
 F 1 "5V" H 800 2100 50  0000 C CNN
-F 2 "" H 800 2000 50  0000 C CNN
+F 2 "conn:CONN_2-SIL" H 800 2000 50  0001 C CNN
 F 3 "" H 800 2000 50  0000 C CNN
 	1    800  2000
@@
 F 0 "Q1" V 1600 2050 50  0000 C CNN
 F 1 "PMV160UP" V 1500 2050 50  0000 C CNN
-F 2 "" H 1350 2050 60  0000 C CNN
+F 2 "IPC-semi-nominal:SOT-23" H 1350 2050 60  0001 C CNN
 F 3 "" H 1350 2050 60  0000 C CNN
 	1    1350 2050
@@
 F 0 "J7" H 10100 3750 50  0000 C CNN
 F 1 "5V" H 10100 3650 50  0000 C CNN
-F 2 "" H 10100 3550 50  0000 C CNN
+F 2 "conn:CONN_2-SIL" H 10100 3550 50  0001 C CNN
 F 3 "" H 10100 3550 50  0000 C CNN
 	1    10100 3550
@@
 F 0 "R5" V 8400 3550 50  0000 C CNN
 F 1 "49r9" V 8500 3550 50  0000 C CNN
-F 2 "" H 8600 3600 60  0000 C CNN
+F 2 "IPC7351-Nominal:RESC1005X40" H 8600 3600 60  0001 C CNN
 F 3 "" H 8600 3600 60  0000 C CNN
 	1    8600 3550
@@
 F 0 "R6" V 9500 3550 50  0000 C CNN
 F 1 "49r9" V 9600 3550 50  0000 C CNN
-F 2 "" H 9700 3600 60  0000 C CNN
+F 2 "IPC7351-Nominal:RESC1005X40" H 9700 3600 60  0001 C CNN
 F 3 "" H 9700 3600 60  0000 C CNN
 	1    9700 3550
@@
 F 0 "C11" H 9600 3850 50  0000 C CNN
 F 1 "1n" H 9600 3750 50  0000 C CNN
-F 2 "" H 9390 3775 60  0000 C CNN
+F 2 "IPC7351-Nominal:CAPC1005X55" H 9390 3775 60  0001 C CNN
 F 3 "" H 9390 3775 60  0000 C CNN
 	1    9400 3800
@@
 F 0 "C10" H 9000 3850 50  0000 C CNN
 F 1 "1n" H 9000 3750 50  0000 C CNN
-F 2 "" H 8790 3775 60  0000 C CNN
+F 2 "IPC7351-Nominal:CAPC1005X55" H 8790 3775 60  0001 C CNN
 F 3 "" H 8790 3775 60  0000 C CNN
 	1    8800 3800
@@
 F 0 "MP1" H 2350 5000 50  0000 C CNN
 F 1 "SHIELD" H 2350 4900 50  0000 C CNN
-F 2 "" H 2350 4800 50  0000 C CNN
+F 2 "" H 2350 4800 50  0001 C CNN
 F 3 "" H 2350 4800 50  0000 C CNN
 	1    2350 4800
@@
 F 0 "J3" H 800 3500 50  0000 C CNN
 F 1 "IN1" H 800 3400 50  0000 C CNN
-F 2 "" H 800 3300 50  0000 C CNN
+F 2 "conn:CONN-2_CONSMA001-SMD-G" H 800 3300 50  0001 C CNN
 F 3 "" H 800 3300 50  0000 C CNN
 	1    800  3300
@@
 F 0 "J2" H 800 2850 50  0000 C CNN
 F 1 "-5V" H 800 2750 50  0000 C CNN
-F 2 "" H 800 2650 50  0000 C CNN
+F 2 "conn:CONN_2-SIL" H 800 2650 50  0001 C CNN
 F 3 "" H 800 2650 50  0000 C CNN
 	1    800  2650
@@
 F 0 "E2" H 1900 2400 50  0000 C CNN
 F 1 "600" H 1900 2500 50  0000 C CNN
-F 2 "" H 1900 2700 60  0000 C CNN
+F 2 "IPC7351-Nominal:INDC1005X60" H 1900 2700 60  0001 C CNN
 F 3 "" H 1900 2700 60  0000 C CNN
+F 4 "BK1005HS601-T" H 1900 2650 60  0001 C CNN "PN"
+F 5 "Value" H 1900 2650 60  0001 C CNN "Manuf"
 	1    1900 2650
 	1    0    0    1
@@
 F 0 "C2" H 2750 2900 50  0000 C CNN
 F 1 "47u" H 2750 2800 50  0000 C CNN
-F 2 "" H 2490 2825 60  0000 C CNN
+F 2 "IPC7351-Nominal:CAPC3216X70" H 2490 2825 60  0001 C CNN
 F 3 "" H 2490 2825 60  0000 C CNN
 F 4 "GRM31CR61A476ME15L" H 1950 2800 40  0000 C CNN "PN"
@@
 F 0 "Q2" V 1600 2700 50  0000 C CNN
 F 1 "2N7002" V 1500 2700 50  0000 C CNN
-F 2 "" H 1350 2700 60  0000 C CNN
+F 2 "IPC-semi-nominal:SOT-23" H 1350 2700 60  0001 C CNN
 F 3 "" H 1350 2700 60  0000 C CNN
 	1    1350 2700
@@
 F 0 "J5" H 800 5600 50  0000 C CNN
 F 1 "CTRL" H 800 5500 50  0000 C CNN
-F 2 "" H 800 5400 50  0000 C CNN
+F 2 "conn:CONN_2-SIL" H 800 5400 50  0001 C CNN
 F 3 "" H 800 5400 50  0000 C CNN
 	1    800  5400
@@
 F 0 "J6" H 800 6100 50  0000 C CNN
 F 1 "PHASEREF" H 800 6000 50  0000 C CNN
-F 2 "" H 800 5900 50  0000 C CNN
+F 2 "conn:CONN-2_CONSMA001-SMD-G" H 800 5900 50  0001 C CNN
 F 3 "" H 800 5900 50  0000 C CNN
 	1    800  5900
@@
 F 0 "C1" H 2750 2250 50  0000 C CNN
 F 1 "47u" H 2750 2150 50  0000 C CNN
-F 2 "" H 2490 2175 60  0000 C CNN
+F 2 "IPC7351-Nominal:CAPC3216X70" H 2490 2175 60  0001 C CNN
 F 3 "" H 2490 2175 60  0000 C CNN
 F 4 "GRM31CR61A476ME15L" H 1950 2150 40  0000 C CNN "PN"
@@
 Wire Wire Line
 	7000 3550 6750 3550
+$Comp
+L BEAD E1
+U 1 1 545FCF7F
+P 1900 2000
+F 0 "E1" H 1900 1750 50  0000 C CNN
+F 1 "600" H 1900 1850 50  0000 C CNN
+F 2 "IPC7351-Nominal:INDC1005X60" H 1900 2050 60  0001 C CNN
+F 3 "" H 1900 2050 60  0000 C CNN
+F 4 "BK1005HS601-T" H 1900 2000 60  0001 C CNN "PN"
+F 5 "Value" H 1900 2000 60  0001 C CNN "Manuf"
+	1    1900 2000
+	1    0    0    1
+$EndComp
 $EndSCHEMATC
