File: pcb/Buffer_Filter.sch (KiCad schematic (older format))
At the start: 18 parts, among them Q6 MMBT3904, Q7 BFR540, Q8 BFR540

Commit message: Associated parts with footprints
Parts:
- C16: footprint (none) -> IPC7351-Nominal:CAPC1005X55
- C17, C18, C19: footprint (none) -> IPC7351-Nominal:CAPC1608X55
- L1, L2: footprint (none) -> IPC7351-Nominal:INDC1005X60; Manuf (none) -> Value; PN (none) -> ELJ-RF27NGFB
- Q6, Q7, Q8: footprint (none) -> IPC-semi-nominal:SOT-23
- R20, R21, R22, R23, R24, R25, R26, R27, R28: footprint (none) -> IPC7351-Nominal:RESC1005X40
Changed lines of the file:
@@
 F 0 "Q7" H 5050 2750 50  0000 C CNN
 F 1 "BFR540" H 5050 2650 50  0000 C CNN
-F 2 "" H 4750 2700 60  0000 C CNN
+F 2 "IPC-semi-nominal:SOT-23" H 4750 2700 60  0001 C CNN
 F 3 "" H 4750 2700 60  0000 C CNN
 	1    4750 2700
@@
 F 0 "Q8" H 5050 3750 50  0000 C CNN
 F 1 "BFR540" H 5050 3650 50  0000 C CNN
-F 2 "" H 4750 3700 60  0000 C CNN
+F 2 "IPC-semi-nominal:SOT-23" H 4750 3700 60  0001 C CNN
 F 3 "" H 4750 3700 60  0000 C CNN
 	1    4750 3700
@@
 F 0 "R25" H 4950 4150 50  0000 C CNN
 F 1 "22" H 4950 4050 50  0000 C CNN
-F 2 "" H 4800 4150 60  0000 C CNN
+F 2 "IPC7351-Nominal:RESC1005X40" H 4800 4150 60  0001 C CNN
 F 3 "" H 4800 4150 60  0000 C CNN
 	1    4800 4100
@@
 F 0 "Q6" H 4100 3950 50  0000 C CNN
 F 1 "MMBT3904" H 4100 3850 50  0000 C CNN
-F 2 "" H 4600 3900 60  0000 C CNN
+F 2 "IPC-semi-nominal:SOT-23" H 4600 3900 60  0001 C CNN
 F 3 "" H 4600 3900 60  0000 C CNN
 	1    4600 3900
@@
 F 0 "C16" H 4500 4050 50  0000 C CNN
 F 1 "10n" H 4500 3950 50  0000 C CNN
-F 2 "" H 4290 3975 60  0000 C CNN
+F 2 "IPC7351-Nominal:CAPC1005X55" H 4290 3975 60  0001 C CNN
 F 3 "" H 4290 3975 60  0000 C CNN
 	1    4300 4000
@@
 F 0 "R23" H 4450 3550 50  0000 C CNN
 F 1 "1k" H 4450 3450 50  0000 C CNN
-F 2 "" H 4300 3550 60  0000 C CNN
+F 2 "IPC7351-Nominal:RESC1005X40" H 4300 3550 60  0001 C CNN
 F 3 "" H 4300 3550 60  0000 C CNN
 	1    4300 3500
@@
 F 0 "R24" H 4550 2950 50  0000 C CNN
 F 1 "200" H 4550 2850 50  0000 C CNN
-F 2 "" H 4400 2950 60  0000 C CNN
+F 2 "IPC7351-Nominal:RESC1005X40" H 4400 2950 60  0001 C CNN
 F 3 "" H 4400 2950 60  0000 C CNN
 	1    4400 2900
@@
 F 0 "R22" H 4250 2950 50  0000 C CNN
 F 1 "200" H 4250 2850 50  0000 C CNN
-F 2 "" H 4100 2950 60  0000 C CNN
+F 2 "IPC7351-Nominal:RESC1005X40" H 4100 2950 60  0001 C CNN
 F 3 "" H 4100 2950 60  0000 C CNN
 	1    4100 2900
@@
 F 0 "R21" H 3950 2950 50  0000 C CNN
 F 1 "200" H 3950 2850 50  0000 C CNN
-F 2 "" H 3800 2950 60  0000 C CNN
+F 2 "IPC7351-Nominal:RESC1005X40" H 3800 2950 60  0001 C CNN
 F 3 "" H 3800 2950 60  0000 C CNN
 	1    3800 2900
@@
 F 0 "R20" H 3650 2950 50  0000 C CNN
 F 1 "200" H 3650 2850 50  0000 C CNN
-F 2 "" H 3500 2950 60  0000 C CNN
+F 2 "IPC7351-Nominal:RESC1005X40" H 3500 2950 60  0001 C CNN
 F 3 "" H 3500 2950 60  0000 C CNN
 	1    3500 2900
@@
 F 0 "R28" V 5250 3200 50  0000 C CNN
 F 1 "100" V 5350 3200 50  0000 C CNN
-F 2 "" H 5450 3250 60  0000 C CNN
+F 2 "IPC7351-Nominal:RESC1005X40" H 5450 3250 60  0001 C CNN
 F 3 "" H 5450 3250 60  0000 C CNN
 	1    5450 3200
@@
 F 0 "R27" V 5200 2200 50  0000 C CNN
 F 1 "100" V 5300 2200 50  0000 C CNN
-F 2 "" H 5400 2250 60  0000 C CNN
+F 2 "IPC7351-Nominal:RESC1005X40" H 5400 2250 60  0001 C CNN
 F 3 "" H 5400 2250 60  0000 C CNN
 	1    5400 2200
@@
 F 0 "R26" H 5250 2450 50  0000 C CNN
 F 1 "100" H 5250 2350 50  0000 C CNN
-F 2 "" H 5100 2450 60  0000 C CNN
+F 2 "IPC7351-Nominal:RESC1005X40" H 5100 2450 60  0001 C CNN
 F 3 "" H 5100 2450 60  0000 C CNN
 	1    5100 2400
@@
 F 0 "C17" H 6700 3550 50  0000 C CNN
 F 1 "22p 1%" H 6700 3450 50  0000 C CNN
-F 2 "" H 6390 3475 60  0000 C CNN
+F 2 "IPC7351-Nominal:CAPC1608X55" H 6390 3475 60  0001 C CNN
 F 3 "" H 6390 3475 60  0000 C CNN
 F 4 "C1608C0G1H220F080AA" H 6400 3500 60  0001 C CNN "PN"
@@
 F 0 "L1" V 6650 3200 50  0000 C CNN
 F 1 "27n 2%" V 6750 3200 50  0000 C CNN
-F 2 "" H 6850 3250 60  0000 C CNN
+F 2 "IPC7351-Nominal:INDC1005X60" H 6850 3250 60  0001 C CNN
 F 3 "" H 6850 3250 60  0000 C CNN
+F 4 "ELJ-RF27NGFB" H 6850 3200 60  0001 C CNN "PN"
+F 5 "Value" H 6850 3200 60  0001 C CNN "Manuf"
 	1    6850 3200
 	0    1    1    0
@@
 F 0 "C18" H 7600 3550 50  0000 C CNN
 F 1 "33p 1%" H 7600 3450 50  0000 C CNN
-F 2 "" H 7290 3475 60  0000 C CNN
+F 2 "IPC7351-Nominal:CAPC1608X55" H 7290 3475 60  0001 C CNN
 F 3 "" H 7290 3475 60  0000 C CNN
 F 4 "C1608C0G1H330F080AA" H 7300 3500 60  0001 C CNN "PN"
@@
 F 0 "L2" V 7600 3200 50  0000 C CNN
 F 1 "27n 2%" V 7700 3200 50  0000 C CNN
-F 2 "" H 7800 3250 60  0000 C CNN
+F 2 "IPC7351-Nominal:INDC1005X60" H 7800 3250 60  0001 C CNN
 F 3 "" H 7800 3250 60  0000 C CNN
+F 4 "ELJ-RF27NGFB" H 7800 3200 60  0001 C CNN "PN"
+F 5 "Value" H 7800 3200 60  0001 C CNN "Manuf"
 	1    7800 3200
 	0    1    1    0
@@
 F 0 "C19" H 8600 3550 50  0000 C CNN
 F 1 "22p 1%" H 8600 3450 50  0000 C CNN
-F 2 "" H 8290 3475 60  0000 C CNN
+F 2 "IPC7351-Nominal:CAPC1608X55" H 8290 3475 60  0001 C CNN
 F 3 "" H 8290 3475 60  0000 C CNN
 F 4 "C1608C0G1H220F080AA" H 8300 3500 60  0001 C CNN "PN"
