File: pcb/Protection.sch (KiCad schematic (older format))
At the start: 18 parts

Commit message: Replaced clamping diode placeholders
Parts:
- removed D1, D2, D3, D4: DIODE, symbol DIODE
- added DZ1, DZ2, DZ5, DZ6: ESD9L5.0ST5G, symbol ESD9L
- renumbered DZ1 to DZ3, DZ2 to DZ4, DZ3 to DZ7, DZ4 to DZ8
Other:
- note removed: "esd9l5-0st5g"
Changed lines of the file:
@@
 $EndComp
 Connection ~ 2650 2600
-$Comp
-L DIODE D1
-U 1 1 545E7B21
-P 3250 3800
-F 0 "D1" H 3450 3850 50  0000 C CNN
-F 1 "DIODE" H 3450 3750 50  0000 C CNN
-F 2 "" H 3250 3800 60  0000 C CNN
-F 3 "" H 3250 3800 60  0000 C CNN
-	1    3250 3800
-	1    0    0    -1
-$EndComp
-$Comp
-L DIODE D2
-U 1 1 545E7B86
-P 3950 3800
-F 0 "D2" H 4150 3850 50  0000 C CNN
-F 1 "DIODE" H 4150 3750 50  0000 C CNN
-F 2 "" H 3950 3800 60  0000 C CNN
-F 3 "" H 3950 3800 60  0000 C CNN
-	1    3950 3800
-	-1   0    0    1
-$EndComp
 Wire Wire Line
 	3250 3700 3250 3500
@@
 Connection ~ 3600 3500
 $Comp
-L BZX84C DZ1
+L BZX84C DZ3
 U 1 1 545E7BDB
 P 3250 4300
-F 0 "DZ1" H 3500 4350 50  0000 C CNN
-F 1 "BZX84C2V7" H 3500 4250 50  0000 C CNN
+F 0 "DZ3" H 3400 4400 50  0000 C CNN
+F 1 "BZX84C2V7" H 3600 4300 50  0000 C CNN
 F 2 "" H 3250 4300 60  0000 C CNN
 F 3 "" H 3250 4300 60  0000 C CNN
@@
 $EndComp
 $Comp
-L BZX84C DZ2
+L BZX84C DZ4
 U 1 1 545E7CA7
 P 3950 4300
-F 0 "DZ2" H 4200 4350 50  0000 C CNN
-F 1 "BZX84C2V7" H 4200 4250 50  0000 C CNN
+F 0 "DZ4" H 3800 4200 50  0000 C CNN
+F 1 "BZX84C2V7" H 4200 4250 50  0001 C CNN
 F 2 "" H 3950 4300 60  0000 C CNN
 F 3 "" H 3950 4300 60  0000 C CNN
@@
 Connection ~ 3600 4600
 $Comp
-L GND #PWR017
+L GND #PWR20
 U 1 1 545E7D2C
 P 3600 4700
-F 0 "#PWR017" H 3600 4700 30  0001 C CNN
+F 0 "#PWR20" H 3600 4700 30  0001 C CNN
 F 1 "GND" H 3600 4630 30  0001 C CNN
 F 2 "" H 3600 4700 60  0000 C CNN
@@
 Connection ~ 3250 4050
 $Comp
-L +5 #PWR018
+L +5 #PWR19
 U 1 1 545E7E15
 P 2700 3950
-F 0 "#PWR018" H 2700 4000 30  0001 C CNN
+F 0 "#PWR19" H 2700 4000 30  0001 C CNN
 F 1 "+5" H 2700 4050 50  0000 C CNN
 F 2 "" H 2700 3950 60  0000 C CNN
@@
 Connection ~ 3950 4050
 $Comp
-L -5 #PWR019
+L -5 #PWR21
 U 1 1 545E7ECD
 P 4550 4150
-F 0 "#PWR019" H 4550 4100 30  0001 C CNN
+F 0 "#PWR21" H 4550 4100 30  0001 C CNN
 F 1 "-5" H 4550 4050 50  0000 C CNN
 F 2 "" H 4550 4150 60  0000 C CNN
@@
 Wire Wire Line
 	4550 4050 4550 4150
-Text Notes 3700 3450 0    60   ~ 0
-esd9l5-0st5g
 Text HLabel 5700 2600 0    60   Input ~ 0
 IN2
@@
 $EndComp
 Connection ~ 6600 2600
-$Comp
-L DIODE D3
-U 1 1 545E850E
-P 7200 3800
-F 0 "D3" H 7400 3850 50  0000 C CNN
-F 1 "DIODE" H 7400 3750 50  0000 C CNN
-F 2 "" H 7200 3800 60  0000 C CNN
-F 3 "" H 7200 3800 60  0000 C CNN
-	1    7200 3800
-	1    0    0    -1
-$EndComp
-$Comp
-L DIODE D4
-U 1 1 545E8514
-P 7900 3800
-F 0 "D4" H 8100 3850 50  0000 C CNN
-F 1 "DIODE" H 8100 3750 50  0000 C CNN
-F 2 "" H 7900 3800 60  0000 C CNN
-F 3 "" H 7900 3800 60  0000 C CNN
-	1    7900 3800
-	-1   0    0    1
-$EndComp
 Wire Wire Line
 	7200 3700 7200 3500
@@
 Connection ~ 7550 3500
 $Comp
-L BZX84C DZ3
+L BZX84C DZ7
 U 1 1 545E8520
 P 7200 4300
-F 0 "DZ3" H 7450 4350 50  0000 C CNN
-F 1 "BZX84C2V7" H 7450 4250 50  0000 C CNN
+F 0 "DZ7" H 7350 4350 50  0000 C CNN
+F 1 "BZX84C2V7" H 7550 4250 50  0000 C CNN
 F 2 "" H 7200 4300 60  0000 C CNN
 F 3 "" H 7200 4300 60  0000 C CNN
@@
 $EndComp
 $Comp
-L BZX84C DZ4
+L BZX84C DZ8
 U 1 1 545E8526
 P 7900 4300
-F 0 "DZ4" H 8150 4350 50  0000 C CNN
-F 1 "BZX84C2V7" H 8150 4250 50  0000 C CNN
+F 0 "DZ8" H 7750 4250 50  0000 C CNN
+F 1 "BZX84C2V7" H 8150 4250 50  0001 C CNN
 F 2 "" H 7900 4300 60  0000 C CNN
 F 3 "" H 7900 4300 60  0000 C CNN
@@
 Connection ~ 7550 4600
 $Comp
-L GND #PWR020
+L GND #PWR25
 U 1 1 545E8533
 P 7550 4700
-F 0 "#PWR020" H 7550 4700 30  0001 C CNN
+F 0 "#PWR25" H 7550 4700 30  0001 C CNN
 F 1 "GND" H 7550 4630 30  0001 C CNN
 F 2 "" H 7550 4700 60  0000 C CNN
@@
 Connection ~ 7200 4050
 $Comp
-L +5 #PWR021
+L +5 #PWR24
 U 1 1 545E8541
 P 6650 3950
-F 0 "#PWR021" H 6650 4000 30  0001 C CNN
+F 0 "#PWR24" H 6650 4000 30  0001 C CNN
 F 1 "+5" H 6650 4050 50  0000 C CNN
 F 2 "" H 6650 3950 60  0000 C CNN
@@
 Connection ~ 7900 4050
 $Comp
-L -5 #PWR022
+L -5 #PWR26
 U 1 1 545E8551
 P 8500 4150
-F 0 "#PWR022" H 8500 4100 30  0001 C CNN
+F 0 "#PWR26" H 8500 4100 30  0001 C CNN
 F 1 "-5" H 8500 4050 50  0000 C CNN
 F 2 "" H 8500 4150 60  0000 C CNN
@@
 Wire Wire Line
 	8500 4050 8500 4150
-Text Notes 7650 3450 0    60   ~ 0
-esd9l5-0st5g
 Text HLabel 4100 2600 2    60   Output ~ 0
 OUT1
@@
 Connection ~ 7550 2600
 $Comp
-L GND #PWR023
+L GND #PWR23
 U 1 1 545E84FE
 P 6600 3000
-F 0 "#PWR023" H 6600 3000 30  0001 C CNN
+F 0 "#PWR23" H 6600 3000 30  0001 C CNN
 F 1 "GND" H 6600 2930 30  0001 C CNN
 F 2 "" H 6600 3000 60  0000 C CNN
@@
 $EndComp
 $Comp
-L GND #PWR024
+L GND #PWR22
 U 1 1 545E84F7
 P 6100 3000
-F 0 "#PWR024" H 6100 3000 30  0001 C CNN
+F 0 "#PWR22" H 6100 3000 30  0001 C CNN
 F 1 "GND" H 6100 2930 30  0001 C CNN
 F 2 "" H 6100 3000 60  0000 C CNN
@@
 $EndComp
 $Comp
-L GND #PWR025
+L GND #PWR18
 U 1 1 545E7848
 P 2650 3000
-F 0 "#PWR025" H 2650 3000 30  0001 C CNN
+F 0 "#PWR18" H 2650 3000 30  0001 C CNN
 F 1 "GND" H 2650 2930 30  0001 C CNN
 F 2 "" H 2650 3000 60  0000 C CNN
@@
 $EndComp
 $Comp
-L GND #PWR026
+L GND #PWR17
 U 1 1 545E782A
 P 2150 3000
-F 0 "#PWR026" H 2150 3000 30  0001 C CNN
+F 0 "#PWR17" H 2150 3000 30  0001 C CNN
 F 1 "GND" H 2150 2930 30  0001 C CNN
 F 2 "" H 2150 3000 60  0000 C CNN
@@
 	1    0    0    -1
 $EndComp
+$Comp
+L ESD9L DZ1
+U 1 1 545FA6EF
+P 3250 3800
+F 0 "DZ1" H 3400 3750 50  0000 C CNN
+F 1 "ESD9L5.0ST5G" H 3600 3850 50  0000 C CNN
+F 2 "" H 3250 3800 60  0000 C CNN
+F 3 "" H 3250 3800 60  0000 C CNN
+	1    3250 3800
+	1    0    0    1
+$EndComp
+$Comp
+L ESD9L DZ2
+U 1 1 545FA788
+P 3950 3800
+F 0 "DZ2" H 3800 3850 50  0000 C CNN
+F 1 "ESD9L5.0ST5G" H 4150 3750 50  0001 C CNN
+F 2 "" H 3950 3800 60  0000 C CNN
+F 3 "" H 3950 3800 60  0000 C CNN
+	1    3950 3800
+	1    0    0    -1
+$EndComp
+$Comp
+L ESD9L DZ5
+U 1 1 545FB15D
+P 7200 3800
+F 0 "DZ5" H 7350 3750 50  0000 C CNN
+F 1 "ESD9L5.0ST5G" H 7550 3850 50  0000 C CNN
+F 2 "" H 7200 3800 60  0000 C CNN
+F 3 "" H 7200 3800 60  0000 C CNN
+	1    7200 3800
+	1    0    0    1
+$EndComp
+$Comp
+L ESD9L DZ6
+U 1 1 545FB1A6
+P 7900 3800
+F 0 "DZ6" H 7750 3850 50  0000 C CNN
+F 1 "ESD9L5.0ST5G" H 8100 3750 50  0001 C CNN
+F 2 "" H 7900 3800 60  0000 C CNN
+F 3 "" H 7900 3800 60  0000 C CNN
+	1    7900 3800
+	1    0    0    -1
+$EndComp

Commit message: Associated parts with footprints
Parts:
- DZ1, DZ2, DZ5, DZ6: footprint (none) -> IPC-semi-nominal:SOD-923
- DZ3, DZ4, DZ7, DZ8: footprint (none) -> IPC-semi-nominal:SOT-23
- F1, F2, R1, R10, R2, R3, R4, R7, R8, R9: footprint (none) -> IPC7351-Nominal:RESC1005X40
Changed lines of the file:
@@
 F 0 "R1" H 2400 2850 50  0000 C CNN
 F 1 "1k6 1%" H 2400 2750 50  0000 C CNN
-F 2 "" H 2150 2850 60  0000 C CNN
+F 2 "IPC7351-Nominal:RESC1005X40" H 2150 2850 60  0001 C CNN
 F 3 "" H 2150 2850 60  0000 C CNN
 	1    2150 2800
@@
 F 0 "R2" H 2900 2850 50  0000 C CNN
 F 1 "1k6 1%" H 2900 2750 50  0000 C CNN
-F 2 "" H 2650 2850 60  0000 C CNN
+F 2 "IPC7351-Nominal:RESC1005X40" H 2650 2850 60  0001 C CNN
 F 3 "" H 2650 2850 60  0000 C CNN
 	1    2650 2800
@@
 F 0 "F1" V 2650 2600 50  0000 C CNN
 F 1 "50mA" V 2750 2600 50  0000 C CNN
-F 2 "" H 2950 2650 60  0000 C CNN
+F 2 "IPC7351-Nominal:RESC1005X40" H 2950 2650 60  0001 C CNN
 F 3 "" H 2950 2650 60  0000 C CNN
 F 4 "F0402G0R05FNTR" V 2850 2600 40  0000 C CNN "PN"
@@
 F 0 "DZ3" H 3400 4400 50  0000 C CNN
 F 1 "BZX84C2V7" H 3600 4300 50  0000 C CNN
-F 2 "" H 3250 4300 60  0000 C CNN
+F 2 "IPC-semi-nominal:SOT-23" H 3250 4300 60  0001 C CNN
 F 3 "" H 3250 4300 60  0000 C CNN
 	1    3250 4300
@@
 F 0 "DZ4" H 3800 4200 50  0000 C CNN
 F 1 "BZX84C2V7" H 4200 4250 50  0001 C CNN
-F 2 "" H 3950 4300 60  0000 C CNN
+F 2 "IPC-semi-nominal:SOT-23" H 3950 4300 60  0001 C CNN
 F 3 "" H 3950 4300 60  0000 C CNN
 	1    3950 4300
@@
 F 0 "R3" V 2750 4050 50  0000 C CNN
 F 1 "1k" V 2850 4050 50  0000 C CNN
-F 2 "" H 2950 4100 60  0000 C CNN
+F 2 "IPC7351-Nominal:RESC1005X40" H 2950 4100 60  0001 C CNN
 F 3 "" H 2950 4100 60  0000 C CNN
 	1    2950 4050
@@
 F 0 "R4" V 4050 4050 50  0000 C CNN
 F 1 "1k" V 4150 4050 50  0000 C CNN
-F 2 "" H 4250 4100 60  0000 C CNN
+F 2 "IPC7351-Nominal:RESC1005X40" H 4250 4100 60  0001 C CNN
 F 3 "" H 4250 4100 60  0000 C CNN
 	1    4250 4050
@@
 F 0 "R7" H 6350 2850 50  0000 C CNN
 F 1 "1k6 1%" H 6350 2750 50  0000 C CNN
-F 2 "" H 6100 2850 60  0000 C CNN
+F 2 "IPC7351-Nominal:RESC1005X40" H 6100 2850 60  0001 C CNN
 F 3 "" H 6100 2850 60  0000 C CNN
 	1    6100 2800
@@
 F 0 "R8" H 6850 2850 50  0000 C CNN
 F 1 "1k6 1%" H 6850 2750 50  0000 C CNN
-F 2 "" H 6600 2850 60  0000 C CNN
+F 2 "IPC7351-Nominal:RESC1005X40" H 6600 2850 60  0001 C CNN
 F 3 "" H 6600 2850 60  0000 C CNN
 	1    6600 2800
@@
 F 0 "F2" V 6600 2600 50  0000 C CNN
 F 1 "50mA" V 6700 2600 50  0000 C CNN
-F 2 "" H 6900 2650 60  0000 C CNN
+F 2 "IPC7351-Nominal:RESC1005X40" H 6900 2650 60  0001 C CNN
 F 3 "" H 6900 2650 60  0000 C CNN
 F 4 "F0402G0R05FNTR" V 6800 2600 40  0000 C CNN "PN"
@@
 F 0 "DZ7" H 7350 4350 50  0000 C CNN
 F 1 "BZX84C2V7" H 7550 4250 50  0000 C CNN
-F 2 "" H 7200 4300 60  0000 C CNN
+F 2 "IPC-semi-nominal:SOT-23" H 7200 4300 60  0001 C CNN
 F 3 "" H 7200 4300 60  0000 C CNN
 	1    7200 4300
@@
 F 0 "DZ8" H 7750 4250 50  0000 C CNN
 F 1 "BZX84C2V7" H 8150 4250 50  0001 C CNN
-F 2 "" H 7900 4300 60  0000 C CNN
+F 2 "IPC-semi-nominal:SOT-23" H 7900 4300 60  0001 C CNN
 F 3 "" H 7900 4300 60  0000 C CNN
 	1    7900 4300
@@
 F 0 "R9" V 6700 4050 50  0000 C CNN
 F 1 "1k" V 6800 4050 50  0000 C CNN
-F 2 "" H 6900 4100 60  0000 C CNN
+F 2 "IPC7351-Nominal:RESC1005X40" H 6900 4100 60  0001 C CNN
 F 3 "" H 6900 4100 60  0000 C CNN
 	1    6900 4050
@@
 F 0 "R10" V 8000 4050 50  0000 C CNN
 F 1 "1k" V 8100 4050 50  0000 C CNN
-F 2 "" H 8200 4100 60  0000 C CNN
+F 2 "IPC7351-Nominal:RESC1005X40" H 8200 4100 60  0001 C CNN
 F 3 "" H 8200 4100 60  0000 C CNN
 	1    8200 4050
@@
 F 0 "DZ1" H 3400 3750 50  0000 C CNN
 F 1 "ESD9L5.0ST5G" H 3600 3850 50  0000 C CNN
-F 2 "" H 3250 3800 60  0000 C CNN
+F 2 "IPC-semi-nominal:SOD-923" H 3250 3800 60  0001 C CNN
 F 3 "" H 3250 3800 60  0000 C CNN
 	1    3250 3800
@@
 F 0 "DZ2" H 3800 3850 50  0000 C CNN
 F 1 "ESD9L5.0ST5G" H 4150 3750 50  0001 C CNN
-F 2 "" H 3950 3800 60  0000 C CNN
+F 2 "IPC-semi-nominal:SOD-923" H 3950 3800 60  0001 C CNN
 F 3 "" H 3950 3800 60  0000 C CNN
 	1    3950 3800
@@
 F 0 "DZ5" H 7350 3750 50  0000 C CNN
 F 1 "ESD9L5.0ST5G" H 7550 3850 50  0000 C CNN
-F 2 "" H 7200 3800 60  0000 C CNN
+F 2 "IPC-semi-nominal:SOD-923" H 7200 3800 60  0001 C CNN
 F 3 "" H 7200 3800 60  0000 C CNN
 	1    7200 3800
@@
 F 0 "DZ6" H 7750 3850 50  0000 C CNN
 F 1 "ESD9L5.0ST5G" H 8100 3750 50  0001 C CNN
-F 2 "" H 7900 3800 60  0000 C CNN
+F 2 "IPC-semi-nominal:SOD-923" H 7900 3800 60  0001 C CNN
 F 3 "" H 7900 3800 60  0000 C CNN
 	1    7900 3800
