File: pcb/Switching.sch (KiCad schematic (older format))
At the start: 13 parts, among them Q3 MMBT3906, Q4 2N7002, Q5 2N7002, U1 MASWSS0162, U2 MASWSS0162

Commit message: Associated parts with footprints
Parts:
- C3, C4: footprint (none) -> IPC7351-Nominal:CAPC1005X55
- Q3, Q4, Q5: footprint (none) -> IPC-semi-nominal:SOT-23
- R11, R12, R13, R14, R15, R16: footprint (none) -> IPC7351-Nominal:RESC1005X40
- U1, U2: footprint (none) -> IPC7351-Nominal:SOIC127P600X175-8
Changed lines of the file:
@@
 F 0 "U2" H 5300 2300 50  0000 C CNN
 F 1 "MASWSS0162" H 5800 2300 50  0000 C CNN
-F 2 "" H 5600 2800 60  0000 C CNN
+F 2 "IPC7351-Nominal:SOIC127P600X175-8" H 5600 2800 60  0001 C CNN
 F 3 "" H 5600 2800 60  0000 C CNN
 	1    5650 2650
@@
 F 0 "U1" H 5300 1600 50  0000 C CNN
 F 1 "MASWSS0162" H 5800 1600 50  0000 C CNN
-F 2 "" H 5600 2100 60  0000 C CNN
+F 2 "IPC7351-Nominal:SOIC127P600X175-8" H 5600 2100 60  0001 C CNN
 F 3 "" H 5600 2100 60  0000 C CNN
 	1    5650 1950
@@
 F 0 "C4" H 5150 4550 50  0000 C CNN
 F 1 "1n" H 5150 4450 50  0000 C CNN
-F 2 "" H 4940 4475 60  0000 C CNN
+F 2 "IPC7351-Nominal:CAPC1005X55" H 4940 4475 60  0001 C CNN
 F 3 "" H 4940 4475 60  0000 C CNN
 	1    4950 4500
@@
 F 0 "C3" H 4950 4550 50  0000 C CNN
 F 1 "1n" H 4950 4450 50  0000 C CNN
-F 2 "" H 4740 4475 60  0000 C CNN
+F 2 "IPC7351-Nominal:CAPC1005X55" H 4740 4475 60  0001 C CNN
 F 3 "" H 4740 4475 60  0000 C CNN
 	1    4750 4500
@@
 F 0 "R14" V 5500 4200 50  0000 C CNN
 F 1 "220" V 5600 4200 50  0000 C CNN
-F 2 "" H 5700 4250 60  0000 C CNN
+F 2 "IPC7351-Nominal:RESC1005X40" H 5700 4250 60  0001 C CNN
 F 3 "" H 5700 4250 60  0000 C CNN
 	1    5700 4200
@@
 F 0 "R13" V 5200 4300 50  0000 C CNN
 F 1 "220" V 5300 4300 50  0000 C CNN
-F 2 "" H 5450 4350 60  0000 C CNN
+F 2 "IPC7351-Nominal:RESC1005X40" H 5450 4350 60  0001 C CNN
 F 3 "" H 5450 4350 60  0000 C CNN
 	1    5450 4300
@@
 F 0 "R12" H 5000 6150 50  0000 C CNN
 F 1 "10k" H 5000 6050 50  0000 C CNN
-F 2 "" H 4850 6150 60  0000 C CNN
+F 2 "IPC7351-Nominal:RESC1005X40" H 4850 6150 60  0001 C CNN
 F 3 "" H 4850 6150 60  0000 C CNN
 	1    4850 6100
@@
 F 0 "Q3" H 5100 5800 50  0000 C CNN
 F 1 "MMBT3906" H 5100 5700 50  0000 C CNN
-F 2 "" H 4800 5750 60  0000 C CNN
+F 2 "IPC-semi-nominal:SOT-23" H 4800 5750 60  0001 C CNN
 F 3 "" H 4800 5750 60  0000 C CNN
 	1    4800 5750
@@
 F 0 "R11" H 5000 5550 50  0000 C CNN
 F 1 "1k" H 5000 5450 50  0000 C CNN
-F 2 "" H 4850 5550 60  0000 C CNN
+F 2 "IPC7351-Nominal:RESC1005X40" H 4850 5550 60  0001 C CNN
 F 3 "" H 4850 5550 60  0000 C CNN
 	1    4850 5500
@@
 F 0 "Q4" H 6250 5950 50  0000 C CNN
 F 1 "2N7002" H 6350 5850 50  0001 C CNN
-F 2 "" H 6100 5900 60  0000 C CNN
+F 2 "IPC-semi-nominal:SOT-23" H 6100 5900 60  0001 C CNN
 F 3 "" H 6100 5900 60  0000 C CNN
 	1    6100 5900
@@
 F 0 "Q5" H 6800 5950 50  0000 C CNN
 F 1 "2N7002" H 6800 5850 50  0000 C CNN
-F 2 "" H 6550 5900 60  0000 C CNN
+F 2 "IPC-semi-nominal:SOT-23" H 6550 5900 60  0001 C CNN
 F 3 "" H 6550 5900 60  0000 C CNN
 	1    6550 5900
@@
 F 0 "R15" H 6300 4050 50  0000 C CNN
 F 1 "10k" H 6300 3950 50  0000 C CNN
-F 2 "" H 6150 4050 60  0000 C CNN
+F 2 "IPC7351-Nominal:RESC1005X40" H 6150 4050 60  0001 C CNN
 F 3 "" H 6150 4050 60  0000 C CNN
 	1    6150 4000
@@
 F 0 "R16" H 6750 4050 50  0000 C CNN
 F 1 "10k" H 6750 3950 50  0000 C CNN
-F 2 "" H 6600 4050 60  0000 C CNN
+F 2 "IPC7351-Nominal:RESC1005X40" H 6600 4050 60  0001 C CNN
 F 3 "" H 6600 4050 60  0000 C CNN
 	1    6600 4000
